File: Hardware/src/UsbOled.kicad_pcb (KiCad board)
At the start: 2 copper layers, 27.4 x 12 mm, 15 parts, among them J1 ‎USB4085, U1 16F1454

Commit message: Updating tracks
Parts:
- DS2: footprint Medo64:DS OLED 128x32 SPI (4w) -> Medo64:DS OLED 128x32 I2C (4w)
Routing:
- net 5V: track 44.9 -> 35.2 mm
- net GND: track 58.0 -> 58.7 mm
