File: src/UsbOled.kicad_pcb (KiCad board)
At the start: 2 copper layers, 27.4 x 12 mm, 15 parts, among them J1 ‎USB4085, U1 16F1454

Commit message: Minor refactorings
Parts:
- J1: footprint Medo64:J USB C 2.0 (16w) -> Medo64:J USB C 2.0 Receptacle (16w)
- U1: footprint Medo64:U Micro PIC16F1454 (TSSOP-14) -> Medo64:U Micro [PIC16F1454] (TSSOP-14)
